Commit message: minor tweaks to build in noetic

File: vpr_tracking/urdf/dodecahedron_wand.urdf.xacro (robot description, xacro)
@@ -2,5 +2,5 @@
 <robot name="dodec_wand" xmlns:xacro="http://www.ros.org/wiki/xacro">
     <xacro:include filename="aruco_marker.xacro"/>
-    <property name="dodecahedron_length" value="0.1476375"/>
+    <xacro:property name="dodecahedron_length" value="0.1476375"/>
   <material name="gray">
     <color rgba="0.8 0.8 0.8 1.0"/>
